Commit message: divide mesh files of hand-e in two folders

File: robotiq_2f_hande_visualization/urdf/robotiq_hande.urdf (robot description, URDF)
Before this commit: robot robotiq_hande, 4 links, 3 joints
Links:
- link hande_left_finger: geometry collision mesh filename=package://robotiq_2f_hande_visualization/meshes/collision/h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 scale=0.001 0.001 0.001; visual mesh filename=package://robotiq_2f_hande_visualization/meshes/collision/h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 scale=0.001 0.001 0.001
- link hande_right_finger: geometry collision mesh filename=package://robotiq_2f_hande_visualization/meshes/collision/h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 scale=0.001 0.001 0.001; visual mesh filename=package://robotiq_2f_hande_visualization/meshes/collision/h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 scale=0.001 0.001 0.001
- link hande_robotiq_hande_base_link: geometry collision mesh filename=package://robotiq_2f_hande_visualization/meshes/collision/h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 scale=0.001 0.001 0.001; visual mesh filename=package://robotiq_2f_hande_visualization/meshes/collision/h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 scale=0.001 0.001 0.001

Commit message: change models for hande

File: robotiq_2f_hande_visualization/urdf/robotiq_hande.urdf (robot description, URDF)
Before this commit: robot robotiq_hande, 4 links, 3 joints
Links:
- link hande_left_finger: geometry collision mesh filename=package://robotiq_2f_hande_visualization/meshes/collision/l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 scale=0.001 0.001 0.001; visual mesh filename=package://robotiq_2f_hande_visualization/meshes/visual/left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 scale=0.001 0.001 0.001
- link hande_right_finger: geometry collision mesh filename=package://robotiq_2f_hande_visualization/meshes/collision/r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 scale=0.001 0.001 0.001; visual mesh filename=package://robotiq_2f_hande_visualization/meshes/visual/righ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 scale=0.001 0.001 0.001
- link hande_robotiq_hande_base_link: geometry collision mesh filename=package://robotiq_2f_hande_visualization/meshes/collision/b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 scale=0.001 0.001 0.001; visual mesh filename=package://robotiq_2f_hande_visualization/meshes/visual/base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 scale=0.001 0.001 0.001
