Commit message: add hande_description

File: catkin_ws/noetic/src/hande_description/urdf/hande.urdf.xacro (robot description, xacro)
@@ -11,5 +11,5 @@
       <origin rpy="0 0 0" xyz="0 0 0"/>
       <geometry>
-        <mesh filename="package://hande_tutorials/meshes/visual/base_link.stl" scale="0.001 0.001 0.001"/>
+        <mesh filename="package://hande_description/meshes/visual/base_link.stl" scale="0.001 0.001 0.001"/>
       </geometry>
       <material name="">
@@ -20,5 +20,5 @@
       <origin rpy="0 0 0" xyz="0 0 0"/>
       <geometry>
-        <mesh filename="package://hande_tutorials/meshes/collision/base_link.stl" scale="0.001 0.001 0.001"/>
+        <mesh filename="package://hande_description/meshes/collision/base_link.stl" scale="0.001 0.001 0.001"/>
       </geometry>
     </collision>
@@ -38,5 +38,5 @@
       <origin rpy="0 0 0" xyz="0 0 0"/>
       <geometry>
-        <mesh filename="package://hande_tutorials/meshes/visual/left_finger.stl" scale="0.001 0.001 0.001"/>
+        <mesh filename="package://hande_description/meshes/visual/left_finger.stl" scale="0.001 0.001 0.001"/>
       </geometry>
       <material name="">
@@ -47,5 +47,5 @@
       <origin rpy="0 0 0" xyz="0 0 0"/>
       <geometry>
-        <mesh filename="package://hande_tutorials/meshes/collision/left_finger.stl" scale="0.001 0.001 0.001"/>
+        <mesh filename="package://hande_description/meshes/collision/left_finger.stl" scale="0.001 0.001 0.001"/>
       </geometry>
     </collision>
@@ -60,5 +60,5 @@
       <origin rpy="0 0 0" xyz="0 0 0"/>
       <geometry>
-        <mesh filename="package://hande_tutorials/meshes/visual/right_finger.stl" scale="0.001 0.001 0.001"/>
+        <mesh filename="package://hande_description/meshes/visual/right_finger.stl" scale="0.001 0.001 0.001"/>
       </geometry>
       <material name="">
@@ -69,5 +69,5 @@
       <origin rpy="0 0 0" xyz="0 0 0"/>
       <geometry>
-        <mesh filename="package://hande_tutorials/meshes/collision/right_finger.stl" scale="0.001 0.001 0.001"/>
+        <mesh filename="package://hande_description/meshes/collision/right_finger.stl" scale="0.001 0.001 0.001"/>
       </geometry>
     </collision>
