Commit message: refactoring

File: ros2_ws/humble/src/hande_description/gazebo/hande_gazebo.xacro (robot description, xacro)
@@ -2,4 +2,5 @@
 <robot xmlns:xacro="http://www.ros.org/wiki/xacro">
   <xacro:macro name="hande_gazebo" params="robot_name">
+    <xacro:property name="hande_control_share" value="$(find hande_control)" />
     <gazebo>
       <plugin name="gz_ros2_control::GazeboSimROS2ControlPlugin" filename="gz_ros2_control-system">
@@ -7,5 +8,5 @@
         <robot_param_node>robot_state_publisher</robot_param_node>
         <update_rate>100.0</update_rate>
-        <parameters>/ros2_ws/install/hande_control/share/hande_control/config/hande_controllers.yaml</parameters>
+        <parameters>${hande_control_share}/config/hande_controllers.yaml</parameters>
       </plugin>
     </gazebo>

File: ros2_ws/humble/src/hande_description/ros2_control/hande_system_interface.xacro (robot description, xacro)
@@ -2,5 +2,4 @@
 <robot xmlns:xacro="http://www.ros.org/wiki/xacro">
   <xacro:macro name="hande_system_interface" params="robot_name mode">
-    <xacro:property name="hande_control_share" value="$(find hande_control)" />
     <ros2_control name="${robot_name}_system_interface" type="system">
       <xacro:if value="${mode == 'gazebo'}">
